File: pcb/Counter thing.kicad_sch (KiCad schematic)
At the start: 13 parts, among them J1 FTSH-105-01-L-DV-007-K, SW1 B3FS-1015, U1 STM32L010K4T6

Commit message: Update KiCad page titles.
Other:
- title: Mini counter -> Counter Thing
Changed lines of the file:
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@@
 	(paper "A4")
 	(title_block
-		(title "Mini counter")
+		(title "Counter Thing")
 		(rev "A")
 		(company "Max Marrone")
